Commit message: force elbow as positive

File: src/ur5e_bullet/ur_e_description/urdf/ur5e.urdf (robot description, URDF)
Before this commit: robot ur5e, 11 links, 10 joints
Joints:
- joint elbow_joint: limit lower=-3.14159265359 upper=3.14159265359 effort=150.0 velocity=3.14 -> lower=-6.28318530718 upper=6.28318530718 effort=150.0 velocity=3.14

File: src/ur5e_bullet/ur_e_description/urdf/ur5e_with_camera.urdf (robot description, URDF)
Before this commit: robot ur5e, 11 links, 10 joints
Joints:
- joint elbow_joint: limit lower=-3.14159265359 upper=3.14159265359 effort=150.0 velocity=3.14 -> lower=-6.28318530718 upper=6.28318530718 effort=150.0 velocity=3.14

Commit message: status 05.08.2026

File: src/ur5e_bullet/ur_e_description/urdf/ur5e.urdf (robot description, URDF)
Before this commit: robot ur5e, 11 links, 10 joints
Links:
- added link scanner_link, mass 0.1; collision mesh filename=../meshes/scanner-stab.stl; visual mesh filename=../meshes/scanner-stab.stl
Joints:
- added joint scanner_joint: type fixed, parent ee_link, child scanner_link, origin xyz=0 0 0.002 rpy=0 1.57079632679 0
